File: hardware/mixxtape.kicad_pcb (KiCad board)
At the start: 2 copper layers, 100.3 x 63.5 mm, 69 parts, among them J1 USB-C_SMD-TYPE-C-31-M-12_1, J4 TF-SMD_TF-01A, J5 PROG_JIG, SW1 SW-SMD_4P-L5.1-W5.1-P3.70-LS6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, SW2 SW-SMD_4P-L5.1-W5.1-P3.70-LS6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, SW3 SW-SMD_4P-L5.1-W5.1-P3.70-LS6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, SW4 SW-SMD_4P-L5.1-W5.1-P3.70-LS6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, U1 WIFI-SMD_ESP32-WROOM-32E, U2 LGA-8_L4.0-W3.0-R_WMM7040DT0, U3 SOIC-8_L5.3-W5.3-P1.27-LS8.0-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, U4 SOT-223-3_L6.5-W3.4-P2.30-LS7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, U8 SOT-23-5_L3.0-W1.7-P0.95-LS2.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

Commit message: readme
Parts:
- added G***: LOGO, LOGO, F.Cu at (122.8, 88.8)
- added G***: LOGO, LOGO, B.Cu at (80.2, 61.7)
- J4: moved to B.Cu
- moved R9 22.5 mm to (92.0, 40.2), turned to 180 degrees
- moved C27 19.1 mm to (73.0, 64.2), turned to 0 degrees
- moved D25 18.0 mm to (89.2, 69.3)
- moved D29 17.9 mm to (71.3, 69.3)
- moved R3 16.3 mm to (114.0, 38.2), turned to 90 degrees
- moved R4 15.3 mm to (113.0, 45.0)
- moved R5 15.3 mm to (113.0, 43.5)
- moved C8 15.3 mm to (113.5, 40.5)
- moved R6 15.3 mm to (113.0, 42.0)
- moved U8 14.8 mm to (73.0, 61.8)
- moved U3 14.4 mm to (107.5, 41.1)
- moved C9 14.1 mm to (112.2, 37.2), turned to 180 degrees
- moved D11 12.9 mm to (63.8, 51.4), turned to 150 degrees
- moved D23 12.9 mm to (96.7, 67.1), turned to -30 degrees
- moved D12 12.8 mm to (67.1, 54.7), turned to 120 degrees
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Routing:
- net VBUS: track 0.00 -> 268.4 mm, vias 0 -> 16
- net 3V3: track 0.00 -> 254.0 mm, vias 0 -> 7
- net CC2_SENSE: track 0.00 -> 140.9 mm, vias 0 -> 2
- net CC1_SENSE: track 0.00 -> 137.3 mm
- net BTN_REC: track 0.00 -> 94.8 mm, vias 0 -> 5
- net PDM_DATA: track 0.00 -> 66.9 mm, vias 0 -> 6
- net PDM_CLK: track 0.00 -> 66.9 mm, vias 0 -> 6
- net SPI_MOSI: track 0.00 -> 60.0 mm, vias 0 -> 2
- net TAB_SENSE: track 0.00 -> 56.1 mm, vias 0 -> 2
- net SPI_CLK: track 0.00 -> 52.3 mm, vias 0 -> 1
- net EN: track 0.00 -> 52.2 mm, vias 0 -> 2
- net SD_DETECT: track 0.00 -> 52.1 mm, vias 0 -> 3
- net BTN_PLAY: track 0.00 -> 46.9 mm, vias 0 -> 2
- net BTN_MODE: track 0.00 -> 46.1 mm, vias 0 -> 2
- net BTN_TRACK: track 0.00 -> 42.4 mm, vias 0 -> 2
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Other:
- outline, holes or cut-outs redrawn
- board text added: "A"
- board text added: "B"
- board text added: "BT"
- board text added: "Board outline 100.33 x 63.50 mm"
- board text added: "C"
- board text added: "FLASH"
- board text added: "Mic faces UP"
- board text added: "Power Only"
- board text added: "Steven Smethurst @Funvill ABlueStar.com 2026-Sept"
- board text removed: "CORRECTION: the brief specifies an acoustic hole through the"
- board text removed: "DEFERRED: the five decorative guide holes along the bottom edge."
- board text removed: "MECHANICAL ONLY - no components placed, no routing."
- board text removed: "NEEDS CHECK against a physical Norelco case before any copper:"
- board text removed: "Outline traced from Open Music Labs Mixtape Alpha released"
- board text removed: "Print at 1:1, cut it out, put it in a case. Brands vary."
- board text removed: "They never enter a deck, so they are artwork rather than"
- board text removed: "board for a bottom-ported mic. The specified part and every"
- board text removed: "board outline from Open Music Labs Mixtape Alpha (CC) — 100.33 x 63.50 mm"
- board text removed: "confirm with them before distributing derived artwork. The shape"
- board text removed: "gerbers. Their wiki states no licence for the design files;"
- board text removed: "in-stock alternative are TOP-ported, so no hole is drawn. Keep"
- board text removed: "is the compact-cassette form factor, so redrawing it from a"
- board text removed: "measured cassette is a straightforward fallback."
- board text removed: "mechanism, and guessed positions would constrain placement for"
- board text removed: "mic faces UP - keep clear, no hole needed"
- board text removed: "no reason. Add them with the silkscreen artwork."
- board text removed: "reel window dia vs hub-clamp ridges, tab position vs internal"
- board text removed: "ribs, lanyard hole vs the case hinge."
- board text removed: "the mic's top face clear of ribs, labels and fingers instead."
