File: hardware/mixxtape.kicad_pcb (KiCad board)
At the start: 2 copper layers, 99.5 x 63.5 mm, 72 parts, among them J1 USB-C_SMD-TYPE-C-31-M-12_1, J4 TF-SMD_TF-01A, J5 PROG_JIG, SW1 SW-SMD_4P-L5.1-W5.1-P3.70-LS6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, SW2 SW-SMD_4P-L5.1-W5.1-P3.70-LS6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, SW3 SW-SMD_4P-L5.1-W5.1-P3.70-LS6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, SW4 SW-SMD_4P-L5.1-W5.1-P3.70-LS6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, U1 WIFI-SMD_ESP32-WROOM-32E, U2 LGA-8_L4.0-W3.0-R_WMM7040DT0, U3 SOIC-8_L5.3-W5.3-P1.27-LS8.0-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, U4 SOT-223-3_L6.5-W3.4-P2.30-LS7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, U8 SOT-23-5_L3.0-W1.7-P0.95-LS2.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

Commit message: hardware: fix what the regression audit found in my own repairs
The MIC_VDD cut-link was on the wrong branch. I verified it by flood-filling
the net with the neck removed: it splits into R12.2+U2.1 in one cluster and
C7.1 alone in another. Cutting it would have left the microphone POWERED and
stripped its decoupling - the opposite of what the commit claimed, and worse
than not having the feature. The segment that actually feeds the mic is only
0.82 mm long with a via at one end and R12's pad at the other, so there is no
room to do it properly. Removed it: R12 is already a 0402 in series with the
mic supply, and lifting one end isolates the mic completely. The feature was
redundant as well as wrong.

Re-tented six vias I had exposed. The SPI_MOSI one at (90.750, 38.600) was
the only untented via whose near neighbour is a DIFFERENT net - 0.411 mm from
the ESP32's ground land, on the part most likely to be hand-reworked, where a
bridge kills the flash bus with no bodge path. Three more sat 0.24-0.38 mm
from same-net 0402 pads, which is a solder-wicking path at reflow on the mic
supply and the flash clock. The last two were PDM_DATA vias sitting 0.225 mm
of bare copper from their own PDM_CLK partner - I had made exactly this
argument about ground vias in an earlier commit and then done it to PDM. 38
probe points remain, still ample.

Mouse-bite pitch 0.85 -> 1.05 mm. At 0.85 the holes were 0.25 mm edge-to-edge,
below JLCPCB's 0.45 mm NPTH-to-NPTH floor. As milled Edge.Cuts circles that
rule never applied; drilling them brought it into scope and nothing caught it,
because min_hole_to_hole was still 0.25 while 19 other severities were
tightened. Raised to 0.45. Also set min_connection 0.0 -> 0.13:
connection_width had been promoted to error but the constraint was zero, so
the rule was inert - it is the one that would have flagged the 0.1475 mm
cut-link necks.

Added second stitching vias to three of the four F.Cu ground islands that
still hung off the plane by a single vi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
Routing:
- net GND: vias 42 -> 45
Changed lines of the file:
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@@
 		(embedded_fonts no)
 	)
+	(footprint "MOUSEBITE_6"
+		(layer "F.Cu")
+		(at 45.2 35.5)
+		(descr "Six 0.6 mm NPTH perforations along the write-protect tab's break line. These were previously drawn as 0.6 mm circles on Edge.Cuts, i.e. as MILLED features - and JLCPCB's minimum internal routing feature is 1.0 mm (0.8 mm at surcharge), so a 0.6 mm milled circle is below what their router can cut. They would have drawn a DFM query, been silently omitted, or broken a bit. Omitted, the tab is a solid 7.4 mm slab of FR4 and the write-protect feature is dead on every board. As drilled holes 0.6 mm is routine. Placed at x = 45.2, y = 35.5 on the board. PITCH IS 1.05 mm, giving 0.45 mm edge-to-edge between holes: at the original 0.85 mm pitch the gap was 0.25 mm, below JLCPCB's NPTH-to-NPTH minimum. As milled Edge.Cuts circles that rule never applied; drilling them brought it into scope.")
+		(tags "mousebite perforation breakaway NPTH")
+		(property "Reference" "MB1"
+			(at 0 -1.6 0)
+			(layer "F.SilkS")
+			(hide yes)
+			(effects
+				(font
+					(size 1 1)
+					(thickness 0.15)
+				)
+			)
+		)
+		(property "Value" "MOUSEBITE_6"
+			(at 0 1.6 0)
+			(layer "F.Fab")
+			(hide yes)
+			(effects
+				(font
+					(size 1 1)
+					(thickness 0.15)
+				)
+			)
+		)
+		(property "Datasheet" ""
+			(at 0 0 0)
+			(layer "F.Fab")
+			(hide yes)
+			(effects
+				(font
+					(size 1.27 1.27)
+				)
+			)
+		)
+		(property "Description" ""
+			(at 0 0 0)
+			(layer "F.Fab")
+			(hide yes)
+			(effects
+				(font
+					(size 1.27 1.27)
+				)
+			)
+		)
+		(attr exclude_from_pos_files exclude_from_bom allow_missing_courtyard)
+		(duplicate_pad_numbers_are_jumpers no)
+		(fp_line
+			(start -4 -0.6)
+			(end 4 -0.6)
+			(stroke
+				(width 0.05)
+				(type solid)
+			)
+			(layer "F.CrtYd")
+		)
+		(fp_line
+			(start -4 0.6)
+			(end -4 -0.6)
+			(stroke
+				(width 0.05)
+				(type solid)
+			)
+			(layer "F.CrtYd")
+		)
+		(fp_line
+			(start 4 -0.6)
+			(end 4 0.6)
+			(stroke
+				(width 0.05)
+				(type solid)
+			)
+			(layer "F.CrtYd")
+		)
+		(fp_line
+			(start 4 0.6)
+			(end -4 0.6)
+			(stroke
+				(width 0.05)
+				(type solid)
+			)
+			(layer "F.CrtYd")
+		)
+		(pad "" np_thru_hole circle
+			(at -3.2 0)
+			(size 0.6 0.6)
+			(drill 0.6)
+			(layers "*.Cu" "Rescue")
+		)
+		(pad "" np_thru_hole circle
+			(at -2.15 0)
+			(size 0.6 0.6)
+			(drill 0.6)
+			(layers "*.Cu" "Rescue")
+		)
+		(pad "" np_thru_hole circle
+			(at -1.1 0)
+			(size 0.6 0.6)
+			(drill 0.6)
+			(layers "*.Cu" "Rescue")
+		)
+		(pad "" np_thru_hole circle
+			(at 1.1 0)
+			(size 0.6 0.6)
+			(drill 0.6)
+			(layers "*.Cu" "Rescue")
+		)
+		(pad "" np_thru_hole circle
+			(at 2.15 0)
+			(size 0.6 0.6)
+			(drill 0.6)
+			(layers "*.Cu" "Rescue")
+		)
+		(pad "" np_thru_hole circle
+			(at 3.2 0)
+			(size 0.6 0.6)
+			(drill 0.6)
+			(layers "*.Cu" "Rescue")
+		)
+		(embedded_fonts no)
+	)
 	(footprint "C0402"
 		(layer "F.Cu")
@@
 		)
 	)
-	(footprint "MOUSEBITE_6"
-		(layer "F.Cu")
-		(at 45.2 35.5)
-		(descr "Six 0.6 mm NPTH perforations along the write-protect tab's break line. These were previously drawn as 0.6 mm circles on Edge.Cuts, i.e. as MILLED features - and JLCPCB's minimum internal routing feature is 1.0 mm (0.8 mm at surcharge), so a 0.6 mm milled circle is below what their router can cut. They would have drawn a DFM query, been silently omitted, or broken a bit. Omitted, the tab is a solid 7.4 mm slab of FR4 and the write-protect feature is dead on every board. As drilled holes 0.6 mm is routine. Placed at x = 45.2, y = 35.5 on the board.")
-		(tags "mousebite perforation breakaway NPTH")
-		(property "Reference" "MB1"
-			(at 0 -1.6 0)
-			(layer "F.SilkS")
-			(hide yes)
-			(effects
-				(font
-					(size 1 1)
-					(thickness 0.15)
-				)
-			)
-		)
-		(property "Value" "MOUSEBITE_6"
-			(at 0 1.6 0)
-			(layer "F.Fab")
-			(hide yes)
-			(effects
-				(font
-					(size 1 1)
-					(thickness 0.15)
-				)
-			)
-		)
-		(property "Datasheet" ""
-			(at 0 0 0)
-			(layer "F.Fab")
-			(hide yes)
-			(effects
-				(font
-					(size 1.27 1.27)
-				)
-			)
-		)
-		(property "Description" ""
-			(at 0 0 0)
-			(layer "F.Fab")
-			(hide yes)
-			(effects
-				(font
-					(size 1.27 1.27)
-				)
-			)
-		)
-		(attr exclude_from_pos_files exclude_from_bom allow_missing_courtyard)
-		(duplicate_pad_numbers_are_jumpers no)
-		(fp_line
-			(start -4 -0.6)
-			(end 4 -0.6)
-			(stroke
-				(width 0.05)
-				(type solid)
-			)
-			(layer "F.CrtYd")
-		)
-		(fp_line
-			(start -4 0.6)
-			(end -4 -0.6)
-			(stroke
-				(width 0.05)
-				(type solid)
-			)
-			(layer "F.CrtYd")
-		)
-		(fp_line
-			(start 4 -0.6)
-			(end 4 0.6)
-			(stroke
-				(width 0.05)
-				(type solid)
-			)
-			(layer "F.CrtYd")
-		)
-		(fp_line
-			(start 4 0.6)
-			(end -4 0.6)
-			(stroke
-				(width 0.05)
-				(type solid)
-			)
-			(layer "F.CrtYd")
-		)
-		(pad "" np_thru_hole circle
-			(at -3.15 0)
-			(size 0.6 0.6)
-			(drill 0.6)
-			(layers "*.Cu" "Rescue")
-		)
-		(pad "" np_thru_hole circle
-			(at -2.3 0)
-			(size 0.6 0.6)
-			(drill 0.6)
-			(layers "*.Cu" "Rescue")
-		)
-		(pad "" np_thru_hole circle
-			(at -1.45 0)
-			(size 0.6 0.6)
-			(drill 0.6)
-			(layers "*.Cu" "Rescue")
-		)
-		(pad "" np_thru_hole circle
-			(at 1.45 0)
-			(size 0.6 0.6)
-			(drill 0.6)
-			(layers "*.Cu" "Rescue")
-		)
-		(pad "" np_thru_hole circle
-			(at 2.3 0)
-			(size 0.6 0.6)
-			(drill 0.6)
-			(layers "*.Cu" "Rescue")
-		)
-		(pad "" np_thru_hole circle
-			(at 3.15 0)
-			(size 0.6 0.6)
-			(drill 0.6)
-			(layers "*.Cu" "Rescue")
-		)
-		(embedded_fonts no)
-	)
 	(footprint "C0402"
 		(layer "F.Cu")
@@
 		(layer "F.Mask")
 	)
-	(gr_rect
-		(start 126.38 43.27)
-		(end 126.98 43.87)
-		(stroke
-			(width 0)
-			(type default)
-		)
-		(fill yes)
-		(layer "F.Mask")
-	)
-	(gr_rect
-		(start 126.38 44.47)
-		(end 126.98 45.07)
-		(stroke
-			(width 0)
-			(type default)
-		)
-		(fill yes)
-		(layer "F.Mask")
-	)
 	(gr_circle
 		(center 69.797918 36.797918)
@@
 	)
 	(via
+		(at 116.02 87.922)
+		(size 0.6)
+		(drill 0.3)
+		(layers "F.Cu" "B.Cu")
+		(tenting
+			(front yes)
+			(back yes)
+		)
+		(net "GND")
+	)
+	(via
 		(at 124.25 39.75)
 		(size 0.6)
@@
 	)
 	(via
+		(at 99.313 45.262)
+		(size 0.6)
+		(drill 0.3)
+		(layers "F.Cu" "B.Cu")
+		(tenting
+			(front yes)
+			(back yes)
+		)
+		(net "GND")
+	)
+	(via
 		(at 91 70.9)
 		(size 0.6)
@@
 	)
 	(via
+		(at 111.281 36.462)
+		(size 0.6)
+		(drill 0.3)
+		(layers "F.Cu" "B.Cu")
+		(tenting
+			(front yes)
+			(back yes)
+		)
+		(net "GND")
+	)
+	(via
 		(at 110.75 37.25)
 		(size 0.6)
@@
 		(layers "F.Cu" "B.Cu")
 		(tenting
-			(front no)
-			(back no)
+			(front yes)
+			(back yes)
 		)
 		(net "LED_DATA")
@@
 	)
 	(segment
-		(start 126.68 44.75)
-		(end 126.68 44.32)
-		(width 0.2)
-		(layer "F.Cu")
-		(net "MIC_VDD")
-	)
-	(segment
 		(start 127.5 44.75)
 		(end 126.68 44.75)
@@
 	)
 	(segment
-		(start 126.68 44.02)
+		(start 126.68 44.75)
 		(end 126.68 43.59)
 		(width 0.2)
@@
 		(net "MIC_VDD")
 	)
-	(segment
-		(start 126.68 44.32)
-		(end 126.68 44.02)
-		(width 0.15)
-		(layer "F.Cu")
-		(net "MIC_VDD")
-	)
 	(via
 		(at 127.5 44.75)
@@
 		(layers "F.Cu" "B.Cu")
 		(tenting
-			(front no)
-			(back no)
+			(front yes)
+			(back yes)
 		)
 		(net "MIC_VDD")
@@
 		(layers "F.Cu" "B.Cu")
 		(tenting
-			(front no)
-			(back no)
+			(front yes)
+			(back yes)
 		)
 		(net "SPI_MOSI")
@@
 		(layers "F.Cu" "B.Cu")
 		(tenting
-			(front no)
-			(back no)
+			(front yes)
+			(back yes)
 		)
 		(net "SPI_CLK")
@@
 		(layers "F.Cu" "B.Cu")
 		(tenting
-			(front no)
-			(back no)
+			(front yes)
+			(back yes)
 		)
 		(net "PDM_DATA")
@@
 		(layers "F.Cu" "B.Cu")
 		(tenting
-			(front no)
-			(back no)
+			(front yes)
+			(back yes)
 		)
 		(net "PDM_DATA")
