File: hardware/mixxtape.kicad_pcb (KiCad board)
At the start: 2 copper layers, 99.5 x 63.5 mm, 72 parts, among them J1 USB-C_SMD-TYPE-C-31-M-12_1, J4 TF-SMD_TF-01A, J5 PROG_JIG, SW1 SW-SMD_4P-L5.1-W5.1-P3.70-LS6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, SW2 SW-SMD_4P-L5.1-W5.1-P3.70-LS6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, SW3 SW-SMD_4P-L5.1-W5.1-P3.70-LS6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, SW4 SW-SMD_4P-L5.1-W5.1-P3.70-LS6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, U1 WIFI-SMD_ESP32-WROOM-32E, U2 LGA-8_L4.0-W3.0-R_WMM7040DT0, U3 SOIC-8_L5.3-W5.3-P1.27-LS8.0-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, U4 SOT-223-3_L6.5-W3.4-P2.30-LS7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, U8 SOT-23-5_L3.0-W1.7-P0.95-LS2.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

Commit message: re running traces
Parts:
- removed the G*** at (80.2, 61.7)
- moved R7 13.7 mm to (63.1, 40.0), turned to -90 degrees
- moved G*** 9.33 mm to (113.7, 91.0)
- moved R11 2.12 mm to (117.8, 87.2)
- moved R1 1.60 mm to (117.8, 84.8)
- moved R10 1.14 mm to (117.8, 86.0)
- moved C9 1.10 mm to (113.2, 36.7), turned to 0 degrees
- moved R3 0.93 mm to (113.1, 38.0), turned to 180 degrees
- moved R9 0.78 mm to (91.4, 40.7), turned to -90 degrees
- moved C8 0.68 mm to (113.1, 41.0)
- moved R2 0.65 mm to (117.8, 88.4)
- moved C2 0.65 mm to (117.2, 75.1)
- moved R6 0.55 mm to (113.0, 42.5)
- moved C1 0.30 mm to (117.2, 73.2)
- moved R5 0.30 mm to (113.0, 43.8)
- moved R4 0.20 mm to (113.0, 45.2)
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Routing:
- net 3V3: track 257.9 -> 251.9 mm, vias 6 -> 5
- net TAB_SENSE: track 56.1 -> 52.0 mm
- net BTN_TRACK: track 42.4 -> 44.7 mm
- net LD24: track 11.5 -> 12.6 mm
- net CC2: track 18.5 -> 17.4 mm
- net VBUS: track 265.7 -> 264.7 mm
- net EN: track 52.2 -> 51.3 mm
- net CC2_SENSE: track 129.7 -> 128.9 mm
- net FLASH_HOLD_N: track 7.95 -> 8.63 mm
- net SPI_MOSI: track 60.0 -> 59.5 mm
- net GND: vias 45 -> 44
